Commit message: Restructure project with src/ folder and ROS2 package

File: src/arm/urdf/left.urdf (robot description, URDF)
Before this commit: robot wujihand-left-v1.0.0, 26 links, 25 joints
Links:
- link finger1_link1: geometry collision mesh filename=package://arm/meshes/left/finger1_link1.STL; visual mesh filename=package://arm/meshes/left/finger1_link1.STL
- link finger1_link2: geometry collision mesh filename=package://arm/meshes/left/finger1_link2.STL; visual mesh filename=package://arm/meshes/left/finger1_link2.STL
- link finger1_link3: geometry collision mesh filename=package://arm/meshes/left/finger1_link3.STL; visual mesh filename=package://arm/meshes/left/finger1_link3.STL
- link finger1_link4: geometry collision mesh filename=package://arm/meshes/left/finger1_link4.STL; visual mesh filename=package://arm/meshes/left/finger1_link4.STL
- link finger1_tip_link: geometry collision mesh filename=package://arm/meshes/left/finger1_tip_link.STL; visual mesh filename=package://arm/meshes/left/finger1_tip_link.STL
- link finger2_link1: geometry collision mesh filename=package://arm/meshes/left/finger2_link1.STL; visual mesh filename=package://arm/meshes/left/finger2_link1.STL
- link finger2_link2: geometry collision mesh filename=package://arm/meshes/left/finger2_link2.STL; visual mesh filename=package://arm/meshes/left/finger2_link2.STL
- link finger2_link3: geometry collision mesh filename=package://arm/meshes/left/finger2_link3.STL; visual mesh filename=package://arm/meshes/left/finger2_link3.STL
- link finger2_link4: geometry collision mesh filename=package://arm/meshes/left/finger2_link4.STL; visual mesh filename=package://arm/meshes/left/finger2_link4.STL
- link finger2_tip_link: geometry collision mesh filename=package://arm/meshes/left/finger2_tip_link.STL; visual mesh filename=package://arm/meshes/left/finger2_tip_link.STL
- link finger3_link1: geometry collision mesh filename=package://arm/meshes/left/finger3_link1.STL; visual mesh filename=package://arm/meshes/left/finger3_link1.STL
- link finger3_link2: geometry collision mesh filename=package://arm/meshes/left/finger3_link2.STL; visual mesh filename=package://arm/meshes/left/finger3_link2.STL
- link finger3_link3: geometry collision mesh filename=package://arm/meshes/left/finger3_link3.STL; visual mesh filename=package://arm/meshes/left/finger3_link3.STL
- link finger3_link4: geometry collision mesh filename=package://arm/meshes/left/finger3_link4.STL; visual mesh filename=package://arm/meshes/left/finger3_link4.STL
- link finger3_tip_link: geometry collision mesh filename=package://arm/meshes/left/finger3_tip_link.STL; visual mesh filename=package://arm/meshes/left/finger3_tip_link.STL
- link finger4_link1: geometry collision mesh filename=package://arm/meshes/left/finger4_link1.STL; visual mesh filename=package://arm/meshes/left/finger4_link1.STL
- link finger4_link2: geometry collision mesh filename=package://arm/meshes/left/finger4_link2.STL; visual mesh filename=package://arm/meshes/left/finger4_link2.STL
- link finger4_link3: geometry collision mesh filename=package://arm/meshes/left/finger4_link3.STL; visual mesh filename=package://arm/meshes/left/finger4_link3.STL
- link finger4_link4: geometry collision mesh filename=package://arm/meshes/left/finger4_link4.STL; visual mesh filename=package://arm/meshes/left/finger4_link4.STL
- link finger4_tip_link: geometry collision mesh filename=package://arm/meshes/left/finger4_tip_link.STL; visual mesh filename=package://arm/meshes/left/finger4_tip_link.STL
- link finger5_link1: geometry collision mesh filename=package://arm/meshes/left/finger5_link1.STL; visual mesh filename=package://arm/meshes/left/finger5_link1.STL
- link finger5_link2: geometry collision mesh filename=package://arm/meshes/left/finger5_link2.STL; visual mesh filename=package://arm/meshes/left/finger5_link2.STL
- link finger5_link3: geometry collision mesh filename=package://arm/meshes/left/finger5_link3.STL; visual mesh filename=package://arm/meshes/left/finger5_link3.STL
- link finger5_link4: geometry collision mesh filename=package://arm/meshes/left/finger5_link4.STL; visual mesh filename=package://arm/meshes/left/finger5_link4.STL
- link finger5_tip_link: geometry collision mesh filename=package://arm/meshes/left/finger5_tip_link.STL; visual mesh filename=package://arm/meshes/left/finger5_tip_link.STL
- link palm_link: geometry collision mesh filename=package://arm/meshes/left/palm_link.STL; visual mesh filename=package://arm/meshes/left/palm_link.STL

Commit message: add more files

File: src/arm/urdf/left.urdf (robot description, URDF)
Before this commit: robot wujihand-left-v1.0.0, 26 links, 25 joints
Links:
- added link base_link; visual box size=0.1 0.1 0.01; visual cylinder length=0.5 radius=0.01
- added link elbow_rot_link
- added link forearm_link; visual cylinder length=0.18 radius=0.02; visual sphere radius=0.02
- added link shoulder_pan_link
- added link upper_arm_link; visual cylinder length=0.2 radius=0.02; visual sphere radius=0.02
- added link wrist_abd_link
- link finger1_link1: mass 0.0075 -> None; geometry visual mesh filename=package://arm/meshes/left/finger1_link1.STL
- link finger1_link2: mass 0.0248 -> None; geometry visual mesh filename=package://arm/meshes/left/finger1_link2.STL
- link finger1_link3: mass 0.0165 -> None; geometry visual mesh filename=package://arm/meshes/left/finger1_link3.STL
- link finger1_link4: mass 0.0165 -> None; geometry visual mesh filename=package://arm/meshes/left/finger1_link4.STL
- link finger1_tip_link: mass 0.004 -> None; geometry visual mesh filename=package://arm/meshes/left/finger1_tip_link.STL
- link finger2_link1: mass 0.0032 -> None; geometry visual mesh filename=package://arm/meshes/left/finger2_link1.STL
- link finger2_link2: mass 0.033 -> None; geometry visual mesh filename=package://arm/meshes/left/finger2_link2.STL
- link finger2_link3: mass 0.0165 -> None; geometry visual mesh filename=package://arm/meshes/left/finger2_link3.STL
- link finger2_link4: mass 0.014 -> None; geometry visual mesh filename=package://arm/meshes/left/finger2_link4.STL
- link finger2_tip_link: mass 0.004 -> None; geometry visual mesh filename=package://arm/meshes/left/finger2_tip_link.STL
- link finger3_link1: mass 0.0032 -> None; geometry visual mesh filename=package://arm/meshes/left/finger3_link1.STL
- link finger3_link2: mass 0.033 -> None; geometry visual mesh filename=package://arm/meshes/left/finger3_link2.STL
- link finger3_link3: mass 0.0165 -> None; geometry visual mesh filename=package://arm/meshes/left/finger3_link3.STL
- link finger3_link4: mass 0.014 -> None; geometry visual mesh filename=package://arm/meshes/left/finger3_link4.STL
- link finger3_tip_link: mass 0.004 -> None; geometry visual mesh filename=package://arm/meshes/left/finger3_tip_link.STL
- link finger4_link1: mass 0.0032 -> None; geometry visual mesh filename=package://arm/meshes/left/finger4_link1.STL
- link finger4_link2: mass 0.033 -> None; geometry visual mesh filename=package://arm/meshes/left/finger4_link2.STL
- link finger4_link3: mass 0.0165 -> None; geometry visual mesh filename=package://arm/meshes/left/finger4_link3.STL
- link finger4_link4: mass 0.014 -> None; geometry visual mesh filename=package://arm/meshes/left/finger4_link4.STL
- link finger4_tip_link: mass 0.004 -> None; geometry visual mesh filename=package://arm/meshes/left/finger4_tip_link.STL
- link finger5_link1: mass 0.0032 -> None; geometry visual mesh filename=package://arm/meshes/left/finger5_link1.STL
- link finger5_link2: mass 0.033 -> None; geometry visual mesh filename=package://arm/meshes/left/finger5_link2.STL
- link finger5_link3: mass 0.0165 -> None; geometry visual mesh filename=package://arm/meshes/left/finger5_link3.STL
- link finger5_link4: mass 0.014 -> None; geometry visual mesh filename=package://arm/meshes/left/finger5_link4.STL
- link finger5_tip_link: mass 0.004 -> None; geometry visual mesh filename=package://arm/meshes/left/finger5_tip_link.STL
Joints:
- added joint elbow_flex_joint: type revolute, parent upper_arm_link, child elbow_rot_link, origin xyz=0.22 0 0 rpy=0 0 0, axis 0 -1 0, limit lower=0 upper=2.6 effort=100 velocity=1.0
- added joint elbow_rot_joint: type revolute, parent elbow_rot_link, child forearm_link, origin xyz=0 0 0 rpy=0 0 0, axis 1 0 0, limit lower=-1.57 upper=1.57 effort=50 velocity=1.5
- added joint shoulder_pan_joint: type revolute, parent base_link, child shoulder_pan_link, origin xyz=0 0 0.5 rpy=0 0 0, axis 0 0 1, limit lower=-1.57 upper=1.57 effort=100 velocity=1.0
- added joint shoulder_tilt_joint: type revolute, parent shoulder_pan_link, child upper_arm_link, origin xyz=0 0 0 rpy=0 0 0, axis 0 1 0, limit lower=-1.57 upper=0.94 effort=100 velocity=1.0
- added joint wrist_abd_joint: type revolute, parent wrist_abd_link, child palm_link, origin xyz=0 0 0 rpy=0 -1.5708 0, axis 0 0 1, limit lower=-2.0 upper=2.0 effort=30 velocity=1.0
- added joint wrist_flex_joint: type revolute, parent forearm_link, child wrist_abd_link, origin xyz=0.19 0 0 rpy=0 0 0, axis 0 1 0, limit lower=1.57 upper=4.71 effort=30 velocity=1.0
- joint finger1_joint1: axis -0 1 -0 -> 0 1 0; limit lower=-0.0448 upper=1.6508 effort=0.6 velocity=8.58701992 -> lower=-0.0448 upper=1.6508 effort=0.6 velocity=8.58
- joint finger1_joint2: limit lower=-0.1659 upper=0.9339 effort=0.6 velocity=11.10029404 -> lower=-0.1659 upper=0.9339 effort=0.6 velocity=11.1
- joint finger1_joint3: limit lower=-0.4932 upper=1.6272 effort=0.3 velocity=12.86307659 -> lower=-0.4932 upper=1.6272 effort=0.3 velocity=12.86
- joint finger1_joint4: limit lower=-0.4932 upper=1.6272 effort=0.3 velocity=13.57866158 -> lower=-0.4932 upper=1.6272 effort=0.3 velocity=13.57
- joint finger1_tip_fixed: axis 0 0 0 -> (none); limit lower=-0.5236 upper=0.5236 effort=100 velocity=10 -> (none)
- joint finger2_joint1: limit lower=-0.32695 upper=1.63595 effort=1 velocity=8.203047484 -> lower=-0.32695 upper=1.63595 effort=1 velocity=8.2
- joint finger2_joint2: axis -1 -0 -0 -> -1 0 0; limit lower=-0.495 upper=0.495 effort=0.2 velocity=8.115781022 -> lower=-0.495 upper=0.495 effort=0.2 velocity=8.11
- joint finger2_joint3: axis -0 1 -0 -> 0 1 0; limit lower=-0.4932 upper=1.6272 effort=0.3 velocity=12.86307659 -> lower=-0.4932 upper=1.6272 effort=0.3 velocity=12.86
- joint finger2_joint4: axis -0 1 -0 -> 0 1 0; limit lower=-0.4932 upper=1.6272 effort=0.3 velocity=13.57866158 -> lower=-0.4932 upper=1.6272 effort=0.3 velocity=13.57
- joint finger2_tip_fixed: axis 0 0 0 -> (none)
- joint finger3_joint1: axis -0 1 -0 -> 0 1 0; limit lower=-0.32695 upper=1.63595 effort=1 velocity=8.203047484 -> lower=-0.32695 upper=1.63595 effort=1 velocity=8.2
- joint finger3_joint2: limit lower=-0.495 upper=0.495 effort=0.2 velocity=8.115781022 -> lower=-0.495 upper=0.495 effort=0.2 velocity=8.11
- joint finger3_joint3: axis -0 1 -0 -> 0 1 0; limit lower=-0.4932 upper=1.6272 effort=0.3 velocity=12.86307659 -> lower=-0.4932 upper=1.6272 effort=0.3 velocity=12.86
- joint finger3_joint4: axis -0 1 -0 -> 0 1 0; limit lower=-0.4932 upper=1.6272 effort=0.3 velocity=13.57866158 -> lower=-0.4932 upper=1.6272 effort=0.3 velocity=13.57
- joint finger3_tip_fixed: axis 0 0 0 -> (none)
- joint finger4_joint1: axis -0 1 -0 -> 0 1 0; limit lower=-0.32695 upper=1.63595 effort=1 velocity=8.203047484 -> lower=-0.32695 upper=1.63595 effort=1 velocity=8.2
- joint finger4_joint2: limit lower=-0.495 upper=0.495 effort=0.2 velocity=8.115781022 -> lower=-0.495 upper=0.495 effort=0.2 velocity=8.11
- joint finger4_joint3: axis -0 1 -0 -> 0 1 0; limit lower=-0.4932 upper=1.6272 effort=0.3 velocity=12.86307659 -> lower=-0.4932 upper=1.6272 effort=0.3 velocity=12.86
- joint finger4_joint4: axis -0 1 -0 -> 0 1 0; limit lower=-0.4932 upper=1.6272 effort=0.3 velocity=13.57866158 -> lower=-0.4932 upper=1.6272 effort=0.3 velocity=13.57
- joint finger4_tip_fixed: axis 0 0 0 -> (none)
- joint finger5_joint1: limit lower=-0.32695 upper=1.63595 effort=1 velocity=8.203047484 -> lower=-0.32695 upper=1.63595 effort=1 velocity=8.2
- joint finger5_joint2: limit lower=-0.495 upper=0.495 effort=0.2 velocity=8.115781022 -> lower=-0.495 upper=0.495 effort=0.2 velocity=8.11
- joint finger5_joint3: axis -0 1 -0 -> 0 1 0; limit lower=-0.4932 upper=1.6272 effort=0.3 velocity=12.86307659 -> lower=-0.4932 upper=1.6272 effort=0.3 velocity=12.86
- joint finger5_joint4: axis -0 1 -0 -> 0 1 0; limit lower=-0.4932 upper=1.6272 effort=0.3 velocity=13.57866158 -> lower=-0.4932 upper=1.6272 effort=0.3 velocity=13.57
- joint finger5_tip_fixed: axis 0 0 0 -> (none); limit effort=100 velocity=10 -> (none)
